File: electrium-esc-v2/MotorDriver.kicad_sch (KiCad schematic)
At the start: 14 parts, among them U1 DRV8323HRTAR

Commit message: Add all connections
Parts:
- added C24: 0.1u, symbol Device:C
- added R15: 10k, symbol Device:R
Connections:
- net V_DRAIN is gone; now on net PWR_SRC: U1.5 (VDRAIN)
- net +3.3V: now also R15.2
- net GND: now also C22.2, C24.2
- net PWR_SRC: now also C22.1, C24.1; no longer C22.2
- net at C20.1, U1.3 (VCP): no longer C22.1
- net CAL: no longer names the net of U1.31 (CAL)
- net CAL: now also R15.1
- net GAIN: no longer names the net of R8.1, R?.2, U1.29 (GAIN)
- net VDS: no longer names the net of R12.1, R14.2, U1.28 (VDS)
Other:
- moved on the sheet: C18, C22
