File: electrium-esc-v2/MCU.kicad_sch (KiCad schematic)
At the start: 27 parts, among them J1 USB_B_Micro, J2 Conn_01x02, U1 NCP1117-3.3_SOT223, U2 W25Q128JVS, U3 RP2040, Y1 ABLS-12.000MHZ-B4-T

Commit message: Add all connections
Parts:
- added C17: 10u, Capacitor_SMD:C_0805_2012Metric, symbol Device:C
- added J1: GPIO, symbol Connector_Generic:Conn_01x08
- added J4: Debugger Pins, symbol Connector_Generic:Conn_01x04
Connections:
- net RUN is gone; now on net +3V3: U3.26 (RUN)
- net +3V3: now also C17.1, J4.1 (Pin_1)
- net GND: now also C17.2, J4.3 (Pin_3)
- net SWCLK: now also J4.2 (Pin_2)
- net SWD: now also J4.4 (Pin_4)
- net at U3.11 (GPIO8): now also J1.4 (Pin_4)
- net at U3.12 (GPIO9): now also J1.5 (Pin_5)
- net at U3.13 (GPIO10): now also J1.6 (Pin_6)
- net at U3.14 (GPIO11): now also J1.7 (Pin_7)
- net at U3.15 (GPIO12): now also J1.8 (Pin_8)
- net LED: now reaches U3.16 (GPIO13)
- net NRF_MISO: now reaches U3.2 (GPIO0)
- net OUT_L3: now reaches U3.27 (GPIO16)
- net OUT_H3: now reaches U3.28 (GPIO17)
- net OUT_L2: now reaches U3.29 (GPIO18)
- net NRF_CS: now reaches U3.3 (GPIO1)
- net OUT_H2: now reaches U3.30 (GPIO19)
- net OUT_L1: now reaches U3.31 (GPIO20)
- net OUT_H1: now reaches U3.32 (GPIO21)
- net ENABLE: now reaches U3.34 (GPIO22)
- net IDRIVE: now reaches U3.35 (GPIO23)
- net MODE: now reaches U3.36 (GPIO24)
- net NFAULT: now reaches U3.37 (GPIO25)
- net SENS1: now reaches U3.39 (GPIO27_ADC1)
- net NRF_CLK: now reaches U3.4 (GPIO2)
- net SENS2: now reaches U3.40 (GPIO28_ADC2)
- net SENS3: now reaches U3.41 (GPIO29_ADC3)
- net NRF_MOSI: now reaches U3.5 (GPIO3)
- net NRF_CE: now reaches U3.6 (GPIO4)
- net at U3.7 (GPIO5): now also J1.1 (Pin_1)
- net at U3.8 (GPIO6): now also J1.2 (Pin_2)
- net at U3.9 (GPIO7): now also J1.3 (Pin_3)
Other:
- note added: "Close to pin 44"
- note added: "Close to pin 45"
- note added: "Crystal"
- note added: "Make sure resistors are close to RP2040"
- note added: "SWD"
- note removed: "Make sure C10 is close to pin 44 of RP2040"
- note removed: "Make sure C8 is close to pin 45 of RP2040"
- note removed: "Make sure R3 and R4 are close to RP2040"
- moved on the sheet: C2, C3, R3, R5, Y1

Commit message: Add CAN bus
Parts:
- removed J1: GPIO, symbol Connector_Generic:Conn_01x08
- added J6: GPIO, Connector_PinSocket_2.54mm:PinSocket_1x07_P2.54mm_Vertical, symbol Connector_Generic:Conn_01x07
Connections:
- net +3V3: no longer C10.1, C11.1, C12.1, C13.1, C14.1, C15.1, C16.1, C17.1, C4.1, C9.1, U1.2 (VO), U3.1 (IOVDD), U3.10 (IOVDD), U3.22 (IOVDD), U3.33 (IOVDD), U3.42 (IOVDD), U3.43 (ADC_AVDD), U3.44 (VREG_IN), U3.48 (USB_VDD), U3.49 (IOVDD)
- net LED: now also U3.18 (GPIO15); no longer U3.16 (GPIO13)
- net at U3.7 (GPIO5): now also J6.1 (Pin_1)
- net at U3.8 (GPIO6): now also J6.2 (Pin_2)
- net at U3.9 (GPIO7): now also J6.3 (Pin_3)
- net at U3.11 (GPIO8): now also J6.4 (Pin_4)
- net at U3.12 (GPIO9): now also J6.5 (Pin_5)
- net at U3.13 (GPIO10): now also J6.6 (Pin_6)
- net at U3.14 (GPIO11): now also J6.7 (Pin_7)
- net CANTX: now reaches U3.15 (GPIO12)
- net LBK: now reaches U3.17 (GPIO14)
- new net +3.3V: C10.1, C11.1, C12.1, C13.1, C14.1, C15.1, C16.1, C17.1, C4.1, C9.1, U1.2 (VO), U3.1 (IOVDD), U3.10 (IOVDD), U3.22 (IOVDD), U3.33 (IOVDD), U3.42 (IOVDD), U3.43 (ADC_AVDD), U3.44 (VREG_IN), U3.48 (USB_VDD), U3.49 (IOVDD)
- new net CANRX: U3.16 (GPIO13)
