File: electrium-esc-v2/electrium-esc-v2.kicad_sch (KiCad schematic)
At the start: 4 parts

Commit message: Add all connections
Connections:
- net MCU/LED: now reaches R2.2
Other:
- sheet MCU ports: added ENABLE, IDRIVE, LED, MODE, NFAULT, NRF_CE, NRF_CLK, NRF_CS, NRF_MISO, NRF_MOSI, OUT_H1, OUT_H2, OUT_H3, OUT_L1, OUT_L2, OUT_L3, SENS1, SENS2, SENS3; removed none
- sheet Motor Driver (DRV8323) ports: added ENABLE, IDRIVE, IN_H1, IN_H2, IN_H3, IN_L1, IN_L2, IN_L3, MODE, M_H1, M_H2, M_H3, M_L1, M_L2, M_L3, NFAULT, SENS1, SENS2, SENS3, SH1, SH2, SH3, SN1, SN2, SN3, SP1, SP2, SP3; removed none
- moved on the sheet: D1, D2, R1, R2

Commit message: Add CAN bus
Parts:
- added J5: CAN, symbol Connector_Generic:Conn_01x04
Connections:
- net +3.3V: now also J5.4 (Pin_4)
- net GND: now also J5.1 (Pin_1)
- new net CAN/CANH: J5.3 (Pin_3)
- new net CAN/CANL: J5.2 (Pin_2)
Other:
- added sheet CAN (CAN.kicad_sch)
- sheet MCU ports: added CANRX, CANTX, LBK; removed none
Changed lines of the file:
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@@
+    (stroke (width 0) (type default))
+  )
+  (wire (pts (xy 91.44 106.68) (xy 107.95 106.68))
     (stroke (width 0) (type default))
   )
@@
     (stroke (width 0) (type default))
   )
+  (wire (pts (xy 91.44 104.14) (xy 107.95 104.14))
+    (stroke (width 0) (type default))
+  )
+  (wire (pts (xy 48.26 107.95) (xy 66.04 107.95))
+    (stroke (width 0) (type default))
+  )
+  (wire (pts (xy 91.44 109.22) (xy 107.95 109.22))
+    (stroke (width 0) (type default))
+  )
   (wire (pts (xy 160.02 106.68) (xy 180.34 106.68))
     (stroke (width 0) (type default))
@@
     (stroke (width 0) (type default))
   )
-  (wire (pts (xy 92.71 105.41) (xy 107.95 105.41))
+  (wire (pts (xy 91.44 80.01) (xy 107.95 80.01))
     (stroke (width 0) (type default))
   )
@@
     (stroke (width 0) (type default))
   )
-  (wire (pts (xy 92.71 107.95) (xy 107.95 107.95))
-    (stroke (width 0) (type default))
-  )
-  (wire (pts (xy 92.71 110.49) (xy 107.95 110.49))
+  (wire (pts (xy 91.44 82.55) (xy 107.95 82.55))
+    (stroke (width 0) (type default))
+  )
+  (wire (pts (xy 91.44 85.09) (xy 107.95 85.09))
     (stroke (width 0) (type default))
   )
@@
     (stroke (width 0) (type default))
   )
+  (wire (pts (xy 48.26 105.41) (xy 66.04 105.41))
+    (stroke (width 0) (type default))
+  )
   (wire (pts (xy 160.02 109.22) (xy 180.34 109.22))
     (stroke (width 0) (type default))
@@
     (stroke (width 0) (type default))
   )
-  (wire (pts (xy 92.71 102.87) (xy 107.95 102.87))
-    (stroke (width 0) (type default))
-  )
-  (wire (pts (xy 92.71 100.33) (xy 107.95 100.33))
+  (wire (pts (xy 91.44 77.47) (xy 107.95 77.47))
+    (stroke (width 0) (type default))
+  )
+  (wire (pts (xy 91.44 74.93) (xy 107.95 74.93))
     (stroke (width 0) (type default))
   )
@@
     )
   )
+  (symbol (lib_id "power:+3.3V") (at 48.26 102.87 0) (unit 1)
+    (in_bom yes) (on_board yes) (dnp no) (fields_autoplaced)
+    (property "Reference" "#PWR038" (at 48.26 106.68 0)
+      (effects (font (size 1.27 1.27)) hide)
+    )
+    (property "Value" "+3.3V" (at 48.26 99.06 0)
+      (effects (font (size 1.27 1.27)))
+    )
+    (property "Footprint" "" (at 48.26 102.87 0)
+      (effects (font (size 1.27 1.27)) hide)
+    )
+    (property "Datasheet" "" (at 48.26 102.87 0)
+      (effects (font (size 1.27 1.27)) hide)
+    )
+    (pin "1")
+    (instances
+      (project "electrium-esc-v2"
+        (path "/be00c12c-11fa-42cb-8a0b-46fcd24b2ced"
+          (reference "#PWR038") (unit 1)
+        )
+      )
+    )
+  )
+  (symbol (lib_id "power:GND") (at 48.26 110.49 0) (unit 1)
+    (in_bom yes) (on_board yes) (dnp no) (fields_autoplaced)
+    (property "Reference" "#PWR039" (at 48.26 116.84 0)
+      (effects (font (size 1.27 1.27)) hide)
+    )
+    (property "Value" "GND" (at 48.26 115.57 0)
+      (effects (font (size 1.27 1.27)))
+    )
+    (property "Footprint" "" (at 48.26 110.49 0)
+      (effects (font (size 1.27 1.27)) hide)
+    )
+    (property "Datasheet" "" (at 48.26 110.49 0)
+      (effects (font (size 1.27 1.27)) hide)
+    )
+    (pin "1")
+    (instances
+      (project "electrium-esc-v2"
+        (path "/be00c12c-11fa-42cb-8a0b-46fcd24b2ced"
+          (reference "#PWR039") (unit 1)
+        )
+      )
+    )
+  )
+  (symbol (lib_id "Connector_Generic:Conn_01x04") (at 43.18 107.95 180) (unit 1)
+    (in_bom yes) (on_board yes) (dnp no) (fields_autoplaced)
+    (property "Reference" "J5" (at 43.18 97.79 0)
+      (effects (font (size 1.27 1.27)))
+    )
+    (property "Value" "CAN" (at 43.18 100.33 0)
+      (effects (font (size 1.27 1.27)))
+    )
+    (property "Footprint" "" (at 43.18 107.95 0)
+      (effects (font (size 1.27 1.27)) hide)
+    )
+    (property "Datasheet" "~" (at 43.18 107.95 0)
+      (effects (font (size 1.27 1.27)) hide)
+    )
+    (pin "1")
+    (pin "2")
+    (pin "3")
+    (pin "4")
+    (instances
+      (project "electrium-esc-v2"
+        (path "/be00c12c-11fa-42cb-8a0b-46fcd24b2ced"
+          (reference "J5") (unit 1)
+        )
+      )
+    )
+  )
   (symbol (lib_id "Device:R") (at 134.62 146.05 180) (unit 1)
     (in_bom yes) (on_board yes) (dnp no)
@@
     )
   )
-  (sheet (at 107.95 74.93) (size 52.07 62.23) (fields_autoplaced)
+  (sheet (at 107.95 44.45) (size 52.07 92.71) (fields_autoplaced)
     (stroke (width 0.3) (type solid))
     (fill (color 0 0 0 0.0000))
-    (property "Sheetname" "MCU" (at 107.95 74.1446 0)
+    (property "Sheetname" "MCU" (at 107.95 43.6646 0)
       (effects (font (size 1.27 1.27)) (justify left bottom))
     )
@@
       (effects (font (size 1.27 1.27)) (justify left top))
     )
-    (pin "NRF_CE" output (at 107.95 107.95 180)
-      (effects (font (size 1.27 1.27)) (justify left))
-    )
-    (pin "NRF_CLK" output (at 107.95 100.33 180)
-      (effects (font (size 1.27 1.27)) (justify left))
-    )
-    (pin "NRF_CS" output (at 107.95 110.49 180)
-      (effects (font (size 1.27 1.27)) (justify left))
-    )
-    (pin "NRF_MOSI" output (at 107.95 102.87 180)
-      (effects (font (size 1.27 1.27)) (justify left))
-    )
-    (pin "NRF_MISO" input (at 107.95 105.41 180)
+    (pin "NRF_CE" output (at 107.95 82.55 180)
+      (effects (font (size 1.27 1.27)) (justify left))
+    )
+    (pin "NRF_CLK" output (at 107.95 74.93 180)
+      (effects (font (size 1.27 1.27)) (justify left))
+    )
+    (pin "NRF_CS" output (at 107.95 85.09 180)
+      (effects (font (size 1.27 1.27)) (justify left))
+    )
+    (pin "NRF_MOSI" output (at 107.95 77.47 180)
+      (effects (font (size 1.27 1.27)) (justify left))
+    )
+    (pin "NRF_MISO" input (at 107.95 80.01 180)
       (effects (font (size 1.27 1.27)) (justify left))
     )
@@
       (effects (font (size 1.27 1.27)) (justify left))
     )
+    (pin "CANTX" output (at 107.95 104.14 180)
+      (effects (font (size 1.27 1.27)) (justify left))
+    )
+    (pin "CANRX" input (at 107.95 106.68 180)
+      (effects (font (size 1.27 1.27)) (justify left))
+    )
+    (pin "LBK" output (at 107.95 109.22 180)
+      (effects (font (size 1.27 1.27)) (justify left))
+    )
     (instances
       (project "electrium-esc-v2"
         (path "/be00c12c-11fa-42cb-8a0b-46fcd24b2ced" (page "2"))
+      )
+    )
+  )
+  (sheet (at 66.04 101.6) (size 25.4 10.16) (fields_autoplaced)
+    (stroke (width 0.3) (type solid))
+    (fill (color 0 0 0 0.0000))
+    (property "Sheetname" "CAN" (at 66.04 100.8146 0)
+      (effects (font (size 1.27 1.27)) (justify left bottom))
+    )
+    (property "Sheetfile" "CAN.kicad_sch" (at 66.04 112.4184 0)
+      (effects (font (size 1.27 1.27)) (justify left top))
+    )
+    (pin "CANH" bidirectional (at 66.04 105.41 180)
+      (effects (font (size 1.27 1.27)) (justify left))
+    )
+    (pin "CANTX" input (at 91.44 104.14 0)
+      (effects (font (size 1.27 1.27)) (justify right))
+    )
+    (pin "CANRX" output (at 91.44 106.68 0)
+      (effects (font (size 1.27 1.27)) (justify right))
+    )
+    (pin "LBK" input (at 91.44 109.22 0)
+      (effects (font (size 1.27 1.27)) (justify right))
+    )
+    (pin "CANL" bidirectional (at 66.04 107.95 180)
+      (effects (font (size 1.27 1.27)) (justify left))
+    )
+    (instances
+      (project "electrium-esc-v2"
+        (path "/be00c12c-11fa-42cb-8a0b-46fcd24b2ced" (page "7"))
       )
     )
@@
     )
   )
-  (sheet (at 67.31 95.25) (size 25.4 19.05) (fields_autoplaced)
+  (sheet (at 66.04 69.85) (size 25.4 19.05) (fields_autoplaced)
     (stroke (width 0.3) (type solid))
     (fill (color 0 0 0 0.0000))
-    (property "Sheetname" "NRF_COMM" (at 67.31 94.4646 0)
+    (property "Sheetname" "NRF_COMM" (at 66.04 69.0646 0)
       (effects (font (size 1.27 1.27)) (justify left bottom))
     )
-    (property "Sheetfile" "NRF_COMM.kicad_sch" (at 67.31 114.9584 0)
+    (property "Sheetfile" "NRF_COMM.kicad_sch" (at 66.04 89.5584 0)
       (effects (font (size 1.27 1.27)) (justify left top))
     )
-    (pin "NRF_MOSI" input (at 92.71 102.87 0)
-      (effects (font (size 1.27 1.27)) (justify right))
-    )
-    (pin "NRF_MISO" output (at 92.71 105.41 0)
-      (effects (font (size 1.27 1.27)) (justify right))
-    )
-    (pin "NRF_SCK" input (at 92.71 100.33 0)
-      (effects (font (size 1.27 1.27)) (justify right))
-    )
-    (pin "NRF_CSN" input (at 92.71 110.49 0)
-      (effects (font (size 1.27 1.27)) (justify right))
-    )
-    (pin "NRF_CE" input (at 92.71 107.95 0)
-      (effects (font (size 1.27 1.27)) (justify right))
-    )
+    (pin "NRF_MOSI" input (at 91.44 77.47 0)
+      (effects (font (size 1.27 1.27)) (justify right))
+    )
+    (pin "NRF_MISO" output (at 91.44 80.01 0)
+      (effects (font (size 1.27 1.27)) (justify right))
+    )
+    (pin "NRF_SCK" input (at 91.44 74.93 0)
+      (effects (font (size 1.27 1.27)) (justify right))
+    )
+    (pin "NRF_CSN" input (at 91.44 85.09 0)
+      (effects (font (size 1.27 1.27)) (justify right))
+    )
+    (pin "NRF_CE" input (at 91.44 82.55 0)
+      (effects (font (size 1.27 1.27)) (justify right))
+    )
