File: NRF_COMM.kicad_sch (KiCad schematic)
At the start: 2 parts, among them U1 NRF24L01_Breakout

Commit message: Re-annotate all components
Parts:
- renumbered C1 to C28, U1 to U5
Changed lines of the file:
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@@
   (symbol (lib_id "RF:NRF24L01_Breakout") (at 139.7 100.33 0) (unit 1)
     (in_bom yes) (on_board yes) (dnp no)
-    (property "Reference" "U1" (at 144.78 87.63 0)
+    (property "Reference" "U5" (at 144.78 87.63 0)
       (effects (font (size 1.27 1.27)) (justify left))
     )
@@
       (project "electrium-esc-v2"
         (path "/be00c12c-11fa-42cb-8a0b-46fcd24b2ced/81cbbca5-64b8-44af-87f0-aec946520ae6"
-          (reference "U1") (unit 1)
+          (reference "U5") (unit 1)
         )
       )
       (project "electrium-esc"
         (path "/d277d506-2f4d-497b-a498-1ff059e212d2/9d2b8e53-abda-48f4-a6e0-4b62c24d8218"
-          (reference "U5") (unit 1)
+          (reference "U?") (unit 1)
         )
       )
@@
   (symbol (lib_id "power:GND") (at 146.05 80.01 0) (unit 1)
     (in_bom yes) (on_board yes) (dnp no)
-    (property "Reference" "#PWR03" (at 146.05 86.36 0)
+    (property "Reference" "#PWR051" (at 146.05 86.36 0)
       (effects (font (size 1.27 1.27)) hide)
     )
@@
       (project "electrium-esc-v2"
         (path "/be00c12c-11fa-42cb-8a0b-46fcd24b2ced/81cbbca5-64b8-44af-87f0-aec946520ae6"
-          (reference "#PWR03") (unit 1)
+          (reference "#PWR051") (unit 1)
         )
       )
       (project "electrium-esc"
         (path "/d277d506-2f4d-497b-a498-1ff059e212d2/9d2b8e53-abda-48f4-a6e0-4b62c24d8218"
-          (reference "#PWR072") (unit 1)
+          (reference "#PWR?") (unit 1)
         )
       )
@@
   (symbol (lib_id "Device:C") (at 146.05 76.2 0) (unit 1)
     (in_bom yes) (on_board yes) (dnp no) (fields_autoplaced)
-    (property "Reference" "C1" (at 149.86 74.9299 0)
+    (property "Reference" "C28" (at 149.86 74.9299 0)
       (effects (font (size 1.27 1.27)) (justify left))
     )
@@
       (project "electrium-esc-v2"
         (path "/be00c12c-11fa-42cb-8a0b-46fcd24b2ced/81cbbca5-64b8-44af-87f0-aec946520ae6"
-          (reference "C1") (unit 1)
+          (reference "C28") (unit 1)
         )
       )
       (project "electrium-esc"
         (path "/d277d506-2f4d-497b-a498-1ff059e212d2/9d2b8e53-abda-48f4-a6e0-4b62c24d8218"
-          (reference "C75") (unit 1)
+          (reference "C?") (unit 1)
         )
       )
@@
   (symbol (lib_id "power:+3.3V") (at 139.7 69.85 0) (unit 1)
     (in_bom yes) (on_board yes) (dnp no) (fields_autoplaced)
-    (property "Reference" "#PWR01" (at 139.7 73.66 0)
+    (property "Reference" "#PWR050" (at 139.7 73.66 0)
       (effects (font (size 1.27 1.27)) hide)
     )
@@
       (project "electrium-esc-v2"
         (path "/be00c12c-11fa-42cb-8a0b-46fcd24b2ced/81cbbca5-64b8-44af-87f0-aec946520ae6"
-          (reference "#PWR01") (unit 1)
+          (reference "#PWR050") (unit 1)
         )
       )
       (project "electrium-esc"
         (path "/d277d506-2f4d-497b-a498-1ff059e212d2/9d2b8e53-abda-48f4-a6e0-4b62c24d8218"
-          (reference "#PWR071") (unit 1)
+          (reference "#PWR?") (unit 1)
         )
       )
@@
   (symbol (lib_id "power:GND") (at 139.7 115.57 0) (unit 1)
     (in_bom yes) (on_board yes) (dnp no)
-    (property "Reference" "#PWR02" (at 139.7 121.92 0)
+    (property "Reference" "#PWR052" (at 139.7 121.92 0)
       (effects (font (size 1.27 1.27)) hide)
     )
@@
       (project "electrium-esc-v2"
         (path "/be00c12c-11fa-42cb-8a0b-46fcd24b2ced/81cbbca5-64b8-44af-87f0-aec946520ae6"
-          (reference "#PWR02") (unit 1)
+          (reference "#PWR052") (unit 1)
         )
       )
       (project "electrium-esc"
         (path "/d277d506-2f4d-497b-a498-1ff059e212d2/9d2b8e53-abda-48f4-a6e0-4b62c24d8218"
-          (reference "#PWR073") (unit 1)
+          (reference "#PWR?") (unit 1)
         )
       )

Commit message: Add proper footprints
Parts:
- removed C28: 47u, Capacitor_THT:CP_Radial_D4.0mm_P1.50mm, symbol Device:C
Changed lines of the file:
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@@
 (kicad_sch (version 20230121) (generator eeschema)
   (paper "A4")
-  (junction (at 139.7 71.12) (diameter 0) (color 0 0 0 0)
-  )
   (no_connect (at 127 107.95))
-  (wire (pts (xy 139.7 69.85) (xy 139.7 71.12))
-    (stroke (width 0) (type default))
-  )
-  (wire (pts (xy 146.05 71.12) (xy 146.05 72.39))
-    (stroke (width 0) (type default))
-  )
-  (wire (pts (xy 139.7 71.12) (xy 146.05 71.12))
-    (stroke (width 0) (type default))
-  )
-  (wire (pts (xy 139.7 71.12) (xy 139.7 85.09))
+  (wire (pts (xy 139.7 69.85) (xy 139.7 85.09))
     (stroke (width 0) (type default))
   )
@@
         )
       )
-    )
-  )
-  (symbol (lib_id "power:GND") (at 146.05 80.01 0) (unit 1)
-    (in_bom yes) (on_board yes) (dnp no)
-    (property "Reference" "#PWR051" (at 146.05 86.36 0)
-      (effects (font (size 1.27 1.27)) hide)
-    )
-    (property "Value" "GND" (at 146.05 83.82 0)
-      (effects (font (size 1.27 1.27)))
-    )
-    (property "Footprint" "" (at 146.05 80.01 0)
-      (effects (font (size 1.27 1.27)) hide)
-    )
-    (property "Datasheet" "" (at 146.05 80.01 0)
-      (effects (font (size 1.27 1.27)) hide)
-    )
-    (pin "1")
-    (instances
-      (project "electrium-esc-v2"
-        (path "/be00c12c-11fa-42cb-8a0b-46fcd24b2ced/81cbbca5-64b8-44af-87f0-aec946520ae6"
-          (reference "#PWR051") (unit 1)
-        )
-      )
-      (project "electrium-esc"
-        (path "/d277d506-2f4d-497b-a498-1ff059e212d2/9d2b8e53-abda-48f4-a6e0-4b62c24d8218"
-          (reference "#PWR?") (unit 1)
-        )
-      )
-    )
-  )
-  (symbol (lib_id "Device:C") (at 146.05 76.2 0) (unit 1)
-    (in_bom yes) (on_board yes) (dnp no) (fields_autoplaced)
-    (property "Reference" "C28" (at 149.86 74.9299 0)
-      (effects (font (size 1.27 1.27)) (justify left))
-    )
-    (property "Value" "47u" (at 149.86 77.4699 0)
-      (effects (font (size 1.27 1.27)) (justify left))
-    )
-    (property "Footprint" "Capacitor_THT:CP_Radial_D4.0mm_P1.50mm" (at 147.0152 80.01 0)
-      (effects (font (size 1.27 1.27)) hide)
-    )
-    (property "Datasheet" "~" (at 146.05 76.2 0)
-      (effects (font (size 1.27 1.27)) hide)
-    )
-    (pin "1")
-    (pin "2")
-    (instances
-      (project "electrium-esc-v2"
-        (path "/be00c12c-11fa-42cb-8a0b-46fcd24b2ced/81cbbca5-64b8-44af-87f0-aec946520ae6"
-          (reference "C28") (unit 1)
-        )
-      )
-      (project "electrium-esc"
-        (path "/d277d506-2f4d-497b-a498-1ff059e212d2/9d2b8e53-abda-48f4-a6e0-4b62c24d8218"
-          (reference "C?") (unit 1)
-        )
-      )
