File: _autosave-MotorDriver.kicad_sch (KiCad schematic)
At the start: 16 parts, among them U4 DRV8323HRTAR

Commit message: Add reference changes
Parts:
- U4: footprint QFN50P600X600X80-41N-D -> ext_footprint:QFN50P600X600X80-41N-D
Changed lines of the file:
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@@
       (effects (font (size 1.27 1.27)))
     )
-    (property "Footprint" "QFN50P600X600X80-41N-D" (at 160.02 71.12 0)
+    (property "Footprint" "ext_footprint:QFN50P600X600X80-41N-D" (at 160.02 71.12 0)
       (effects (font (size 1.27 1.27)) (justify left) hide)
     )
