File: buck-convert.kicad_sch (KiCad schematic)
At the start: 10 parts, among them IC1 LMR36510FADDAR

Commit message: Add buck converter
Parts:
- added C31: 3300u, symbol Device:C
- C25: renamed from C26; footprint (none) -> Capacitor_SMD:C_0603_1608Metric
- C26: renamed from C27; footprint (none) -> Capacitor_SMD:C_0603_1608Metric
- C27: renamed from C28; footprint (none) -> Capacitor_SMD:C_0603_1608Metric
- C28: renamed from C?; footprint (none) -> Capacitor_SMD:C_0603_1608Metric
- C29: footprint (none) -> Capacitor_SMD:C_0603_1608Metric
- IC1: footprint SOIC127P600X170-9N -> ext_footprint:SOIC127P600X170-9N
- L1: value 20u -> 22u; footprint (none) -> Inductor_SMD:L_Taiyo-Yuden_NR-30xx
- R17: renamed from R16; footprint (none) -> Resistor_SMD:R_0603_1608Metric
- R18: renamed from R17; footprint (none) -> Resistor_SMD:R_0603_1608Metric
- R19: renamed from R18; footprint (none) -> Resistor_SMD:R_0603_1608Metric
Connections:
- net GND: now also C31.2
- net PWR_SRC: now also C31.1
Changed lines of the file:
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@@
+    (stroke (width 0) (type default))
+  )
+  (wire (pts (xy 181.61 48.26) (xy 185.42 48.26))
     (stroke (width 0) (type default))
   )
@@
     )
   )
+  (global_label "PWR_SRC" (shape input) (at 181.61 48.26 180) (fields_autoplaced)
+    (effects (font (size 1.27 1.27)) (justify right))
+    (property "Intersheetrefs" "${INTERSHEET_REFS}" (at 169.9957 48.26 0)
+      (effects (font (size 1.27 1.27)) (justify right) hide)
+    )
+  )
   (symbol (lib_id "Device:C") (at 119.38 81.28 0) (unit 1)
     (in_bom yes) (on_board yes) (dnp no) (fields_autoplaced)
-    (property "Reference" "C27" (at 123.19 80.645 0)
+    (property "Reference" "C26" (at 123.19 80.645 0)
       (effects (font (size 1.27 1.27)) (justify left))
     )
@@
       (effects (font (size 1.27 1.27)) (justify left))
     )
-    (property "Footprint" "" (at 120.3452 85.09 0)
+    (property "Footprint" "Capacitor_SMD:C_0603_1608Metric" (at 120.3452 85.09 0)
       (effects (font (size 1.27 1.27)) hide)
     )
@@
       (project "electrium-esc-v2"
         (path "/be00c12c-11fa-42cb-8a0b-46fcd24b2ced/dedba472-5e9c-489a-b80e-963af35f7eb6"
-          (reference "C27") (unit 1)
+          (reference "C26") (unit 1)
         )
       )
@@
       (effects (font (size 1.27 1.27)) (justify right))
     )
-    (property "Footprint" "" (at 214.9348 80.01 0)
+    (property "Footprint" "Capacitor_SMD:C_0603_1608Metric" (at 214.9348 80.01 0)
       (effects (font (size 1.27 1.27)) hide)
     )
@@
       (effects (font (size 1.27 1.27)))
     )
-    (property "Footprint" "SOIC127P600X170-9N" (at 161.29 69.85 0)
+    (property "Footprint" "ext_footprint:SOIC127P600X170-9N" (at 161.29 69.85 0)
       (effects (font (size 1.27 1.27)) (justify left) hide)
     )
@@
   (symbol (lib_id "Device:C") (at 171.45 72.39 90) (unit 1)
     (in_bom yes) (on_board yes) (dnp no) (fields_autoplaced)
-    (property "Reference" "C28" (at 171.45 66.04 90)
+    (property "Reference" "C27" (at 171.45 66.04 90)
       (effects (font (size 1.27 1.27)))
     )
@@
       (effects (font (size 1.27 1.27)))
     )
-    (property "Footprint" "" (at 175.26 71.4248 0)
+    (property "Footprint" "Capacitor_SMD:C_0603_1608Metric" (at 175.26 71.4248 0)
       (effects (font (size 1.27 1.27)) hide)
     )
@@
       (project "electrium-esc-v2"
         (path "/be00c12c-11fa-42cb-8a0b-46fcd24b2ced/dedba472-5e9c-489a-b80e-963af35f7eb6"
-          (reference "C28") (unit 1)
+          (reference "C27") (unit 1)
         )
       )
@@
   (symbol (lib_id "power:GND") (at 133.35 67.31 180) (unit 1)
     (in_bom yes) (on_board yes) (dnp no) (fields_autoplaced)
-    (property "Reference" "#PWR040" (at 133.35 60.96 0)
+    (property "Reference" "#PWR038" (at 133.35 60.96 0)
       (effects (font (size 1.27 1.27)) hide)
     )
@@
       (project "electrium-esc-v2"
         (path "/be00c12c-11fa-42cb-8a0b-46fcd24b2ced/dedba472-5e9c-489a-b80e-963af35f7eb6"
-          (reference "#PWR040") (unit 1)
+          (reference "#PWR038") (unit 1)
         )
       )
@@
   (symbol (lib_id "Device:R") (at 173.99 77.47 90) (unit 1)
     (in_bom yes) (on_board yes) (dnp no)
-    (property "Reference" "R16" (at 168.91 76.2 90)
+    (property "Reference" "R17" (at 168.91 76.2 90)
       (effects (font (size 1.27 1.27)))
     )
@@
       (effects (font (size 1.27 1.27)))
     )
-    (property "Footprint" "" (at 173.99 79.248 90)
+    (property "Footprint" "Resistor_SMD:R_0603_1608Metric" (at 173.99 79.248 90)
       (effects (font (size 1.27 1.27)) hide)
     )
@@
       (project "electrium-esc-v2"
         (path "/be00c12c-11fa-42cb-8a0b-46fcd24b2ced/dedba472-5e9c-489a-b80e-963af35f7eb6"
-          (reference "R16") (unit 1)
+          (reference "R17") (unit 1)
         )
       )
@@
   (symbol (lib_id "power:GND") (at 156.21 100.33 0) (unit 1)
     (in_bom yes) (on_board yes) (dnp no) (fields_autoplaced)
-    (property "Reference" "#PWR041" (at 156.21 106.68 0)
+    (property "Reference" "#PWR039" (at 156.21 106.68 0)
       (effects (font (size 1.27 1.27)) hide)
     )
@@
       (project "electrium-esc-v2"
         (path "/be00c12c-11fa-42cb-8a0b-46fcd24b2ced/dedba472-5e9c-489a-b80e-963af35f7eb6"
-          (reference "#PWR041") (unit 1)
+          (reference "#PWR039") (unit 1)
+        )
+      )
+    )
+  )
+  (symbol (lib_id "Device:C") (at 185.42 52.07 0) (unit 1)
+    (in_bom yes) (on_board yes) (dnp no) (fields_autoplaced)
+    (property "Reference" "C31" (at 189.23 51.435 0)
+      (effects (font (size 1.27 1.27)) (justify left))
+    )
+    (property "Value" "3300u" (at 189.23 53.975 0)
+      (effects (font (size 1.27 1.27)) (justify left))
+    )
+    (property "Footprint" "" (at 186.3852 55.88 0)
+      (effects (font (size 1.27 1.27)) hide)
+    )
+    (property "Datasheet" "~" (at 185.42 52.07 0)
+      (effects (font (size 1.27 1.27)) hide)
+    )
+    (pin "1")
+    (pin "2")
+    (instances
+      (project "electrium-esc-v2"
+        (path "/be00c12c-11fa-42cb-8a0b-46fcd24b2ced/dedba472-5e9c-489a-b80e-963af35f7eb6"
+          (reference "C31") (unit 1)
         )
       )
@@
       (effects (font (size 1.27 1.27)))
     )
-    (property "Value" "20u" (at 182.88 73.66 90)
-      (effects (font (size 1.27 1.27)))
-    )
-    (property "Footprint" "" (at 182.88 74.93 0)
+    (property "Value" "22u" (at 182.88 73.66 90)
+      (effects (font (size 1.27 1.27)))
+    )
+    (property "Footprint" "Inductor_SMD:L_Taiyo-Yuden_NR-30xx" (at 182.88 74.93 0)
       (effects (font (size 1.27 1.27)) hide)
     )
@@
   (symbol (lib_id "Device:R") (at 201.93 78.74 0) (unit 1)
     (in_bom yes) (on_board yes) (dnp no) (fields_autoplaced)
-    (property "Reference" "R17" (at 204.47 78.105 0)
+    (property "Reference" "R18" (at 204.47 78.105 0)
       (effects (font (size 1.27 1.27)) (justify left))
     )
@@
       (effects (font (size 1.27 1.27)) (justify left))
     )
-    (property "Footprint" "" (at 200.152 78.74 90)
+    (property "Footprint" "Resistor_SMD:R_0603_1608Metric" (at 200.152 78.74 90)
       (effects (font (size 1.27 1.27)) hide)
     )
@@
       (project "electrium-esc-v2"
         (path "/be00c12c-11fa-42cb-8a0b-46fcd24b2ced/dedba472-5e9c-489a-b80e-963af35f7eb6"
-          (reference "R17") (unit 1)
+          (reference "R18") (unit 1)
         )
       )
@@
   (symbol (lib_id "power:+3.3V") (at 231.14 74.93 0) (unit 1)
     (in_bom yes) (on_board yes) (dnp no) (fields_autoplaced)
-    (property "Reference" "#PWR042" (at 231.14 78.74 0)
+    (property "Reference" "#PWR040" (at 231.14 78.74 0)
       (effects (font (size 1.27 1.27)) hide)
     )
@@
       (project "electrium-esc-v2"
         (path "/be00c12c-11fa-42cb-8a0b-46fcd24b2ced/dedba472-5e9c-489a-b80e-963af35f7eb6"
-          (reference "#PWR042") (unit 1)
+          (reference "#PWR040") (unit 1)
+        )
+      )
+    )
+  )
+  (symbol (lib_id "power:GND") (at 185.42 55.88 0) (unit 1)
+    (in_bom yes) (on_board yes) (dnp no) (fields_autoplaced)
+    (property "Reference" "#PWR043" (at 185.42 62.23 0)
+      (effects (font (size 1.27 1.27)) hide)
+    )
+    (property "Value" "GND" (at 185.42 60.96 0)
+      (effects (font (size 1.27 1.27)))
+    )
+    (property "Footprint" "" (at 185.42 55.88 0)
+      (effects (font (size 1.27 1.27)) hide)
+    )
+    (property "Datasheet" "" (at 185.42 55.88 0)
+      (effects (font (size 1.27 1.27)) hide)
+    )
+    (pin "1")
+    (instances
+      (project "electrium-esc-v2"
+        (path "/be00c12c-11fa-42cb-8a0b-46fcd24b2ced/dedba472-5e9c-489a-b80e-963af35f7eb6"
+          (reference "#PWR043") (unit 1)
         )
       )
@@
   (symbol (lib_id "Device:C") (at 190.5 78.74 180) (unit 1)
     (in_bom yes) (on_board yes) (dnp no) (fields_autoplaced)
-    (property "Reference" "C?" (at 194.31 78.105 0)
+    (property "Reference" "C28" (at 194.31 78.105 0)
       (effects (font (size 1.27 1.27)) (justify right))
     )
@@
       (effects (font (size 1.27 1.27)) (justify right))
     )
-    (property "Footprint" "" (at 189.5348 74.93 0)
+    (property "Footprint" "Capacitor_SMD:C_0603_1608Metric" (at 189.5348 74.93 0)
       (effects (font (size 1.27 1.27)) hide)
     )
@@
       (project "electrium-esc-v2"
         (path "/be00c12c-11fa-42cb-8a0b-46fcd24b2ced/dedba472-5e9c-489a-b80e-963af35f7eb6"
-          (reference "C?") (unit 1)
+          (reference "C28") (unit 1)
         )
       )
@@
   (symbol (lib_id "Device:C") (at 107.95 81.28 0) (unit 1)
     (in_bom yes) (on_board yes) (dnp no) (fields_autoplaced)
-    (property "Reference" "C26" (at 111.76 80.645 0)
+    (property "Reference" "C25" (at 111.76 80.645 0)
       (effects (font (size 1.27 1.27)) (justify left))
     )
@@
       (effects (font (size 1.27 1.27)) (justify left))
     )
-    (property "Footprint" "" (at 108.9152 85.09 0)
+    (property "Footprint" "Capacitor_SMD:C_0603_1608Metric" (at 108.9152 85.09 0)
       (effects (font (size 1.27 1.27)) hide)
     )
@@
       (project "electrium-esc-v2"
         (path "/be00c12c-11fa-42cb-8a0b-46fcd24b2ced/dedba472-5e9c-489a-b80e-963af35f7eb6"
-          (reference "C26") (unit 1)
+          (reference "C25") (unit 1)
         )
       )
@@
   (symbol (lib_id "Device:R") (at 201.93 91.44 0) (unit 1)
     (in_bom yes) (on_board yes) (dnp no) (fields_autoplaced)
-    (property "Reference" "R18" (at 204.47 90.805 0)
+    (property "Reference" "R19" (at 204.47 90.805 0)
       (effects (font (size 1.27 1.27)) (justify left))
     )
@@
       (effects (font (size 1.27 1.27)) (justify left))
     )
-    (property "Footprint" "" (at 200.152 91.44 90)
+    (property "Footprint" "Resistor_SMD:R_0603_1608Metric" (at 200.152 91.44 90)
       (effects (font (size 1.27 1.27)) hide)
     )
@@
       (project "electrium-esc-v2"
         (path "/be00c12c-11fa-42cb-8a0b-46fcd24b2ced/dedba472-5e9c-489a-b80e-963af35f7eb6"
-          (reference "R18") (unit 1)
-        )
-      )
+          (reference "R19") (unit 1)
+        )
+      )

Commit message: Re-annotate all components
Parts:
- renumbered C31 to C29, C27 to C30, C28 to C31, C25 to C32, C26 to C33, C29 to C34, R17 to R13, R18 to R14, R19 to R15
Changed lines of the file:
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@@
   (symbol (lib_id "Device:C") (at 119.38 81.28 0) (unit 1)
     (in_bom yes) (on_board yes) (dnp no) (fields_autoplaced)
-    (property "Reference" "C26" (at 123.19 80.645 0)
+    (property "Reference" "C33" (at 123.19 80.645 0)
       (effects (font (size 1.27 1.27)) (justify left))
     )
@@
       (project "electrium-esc-v2"
         (path "/be00c12c-11fa-42cb-8a0b-46fcd24b2ced/dedba472-5e9c-489a-b80e-963af35f7eb6"
-          (reference "C26") (unit 1)
+          (reference "C33") (unit 1)
         )
       )
@@
   (symbol (lib_id "Device:C") (at 215.9 83.82 180) (unit 1)
     (in_bom yes) (on_board yes) (dnp no) (fields_autoplaced)
-    (property "Reference" "C29" (at 219.71 83.185 0)
+    (property "Reference" "C34" (at 219.71 83.185 0)
       (effects (font (size 1.27 1.27)) (justify right))
     )
@@
       (project "electrium-esc-v2"
         (path "/be00c12c-11fa-42cb-8a0b-46fcd24b2ced/dedba472-5e9c-489a-b80e-963af35f7eb6"
-          (reference "C29") (unit 1)
+          (reference "C34") (unit 1)
         )
       )
@@
   (symbol (lib_id "Device:C") (at 171.45 72.39 90) (unit 1)
     (in_bom yes) (on_board yes) (dnp no) (fields_autoplaced)
-    (property "Reference" "C27" (at 171.45 66.04 90)
+    (property "Reference" "C30" (at 171.45 66.04 90)
       (effects (font (size 1.27 1.27)))
     )
@@
       (project "electrium-esc-v2"
         (path "/be00c12c-11fa-42cb-8a0b-46fcd24b2ced/dedba472-5e9c-489a-b80e-963af35f7eb6"
-          (reference "C27") (unit 1)
+          (reference "C30") (unit 1)
         )
       )
@@
   (symbol (lib_id "power:GND") (at 133.35 67.31 180) (unit 1)
     (in_bom yes) (on_board yes) (dnp no) (fields_autoplaced)
-    (property "Reference" "#PWR038" (at 133.35 60.96 0)
+    (property "Reference" "#PWR047" (at 133.35 60.96 0)
       (effects (font (size 1.27 1.27)) hide)
     )
@@
       (project "electrium-esc-v2"
         (path "/be00c12c-11fa-42cb-8a0b-46fcd24b2ced/dedba472-5e9c-489a-b80e-963af35f7eb6"
-          (reference "#PWR038") (unit 1)
+          (reference "#PWR047") (unit 1)
         )
       )
@@
   (symbol (lib_id "Device:R") (at 173.99 77.47 90) (unit 1)
     (in_bom yes) (on_board yes) (dnp no)
-    (property "Reference" "R17" (at 168.91 76.2 90)
+    (property "Reference" "R13" (at 168.91 76.2 90)
       (effects (font (size 1.27 1.27)))
     )
@@
       (project "electrium-esc-v2"
         (path "/be00c12c-11fa-42cb-8a0b-46fcd24b2ced/dedba472-5e9c-489a-b80e-963af35f7eb6"
-          (reference "R17") (unit 1)
+          (reference "R13") (unit 1)
         )
       )
@@
   (symbol (lib_id "power:GND") (at 156.21 100.33 0) (unit 1)
     (in_bom yes) (on_board yes) (dnp no) (fields_autoplaced)
-    (property "Reference" "#PWR039" (at 156.21 106.68 0)
+    (property "Reference" "#PWR049" (at 156.21 106.68 0)
       (effects (font (size 1.27 1.27)) hide)
     )
@@
       (project "electrium-esc-v2"
         (path "/be00c12c-11fa-42cb-8a0b-46fcd24b2ced/dedba472-5e9c-489a-b80e-963af35f7eb6"
-          (reference "#PWR039") (unit 1)
+          (reference "#PWR049") (unit 1)
         )
       )
@@
   (symbol (lib_id "Device:C") (at 185.42 52.07 0) (unit 1)
     (in_bom yes) (on_board yes) (dnp no) (fields_autoplaced)
-    (property "Reference" "C31" (at 189.23 51.435 0)
+    (property "Reference" "C29" (at 189.23 51.435 0)
       (effects (font (size 1.27 1.27)) (justify left))
     )
@@
       (project "electrium-esc-v2"
         (path "/be00c12c-11fa-42cb-8a0b-46fcd24b2ced/dedba472-5e9c-489a-b80e-963af35f7eb6"
-          (reference "C31") (unit 1)
+          (reference "C29") (unit 1)
         )
       )
@@
   (symbol (lib_id "Device:R") (at 201.93 78.74 0) (unit 1)
     (in_bom yes) (on_board yes) (dnp no) (fields_autoplaced)
-    (property "Reference" "R18" (at 204.47 78.105 0)
+    (property "Reference" "R14" (at 204.47 78.105 0)
       (effects (font (size 1.27 1.27)) (justify left))
     )
@@
       (project "electrium-esc-v2"
         (path "/be00c12c-11fa-42cb-8a0b-46fcd24b2ced/dedba472-5e9c-489a-b80e-963af35f7eb6"
-          (reference "R18") (unit 1)
+          (reference "R14") (unit 1)
         )
       )
@@
   (symbol (lib_id "power:+3.3V") (at 231.14 74.93 0) (unit 1)
     (in_bom yes) (on_board yes) (dnp no) (fields_autoplaced)
-    (property "Reference" "#PWR040" (at 231.14 78.74 0)
+    (property "Reference" "#PWR048" (at 231.14 78.74 0)
       (effects (font (size 1.27 1.27)) hide)
     )
@@
       (project "electrium-esc-v2"
         (path "/be00c12c-11fa-42cb-8a0b-46fcd24b2ced/dedba472-5e9c-489a-b80e-963af35f7eb6"
-          (reference "#PWR040") (unit 1)
+          (reference "#PWR048") (unit 1)
         )
       )
@@
   (symbol (lib_id "power:GND") (at 185.42 55.88 0) (unit 1)
     (in_bom yes) (on_board yes) (dnp no) (fields_autoplaced)
-    (property "Reference" "#PWR043" (at 185.42 62.23 0)
+    (property "Reference" "#PWR046" (at 185.42 62.23 0)
       (effects (font (size 1.27 1.27)) hide)
     )
@@
       (project "electrium-esc-v2"
         (path "/be00c12c-11fa-42cb-8a0b-46fcd24b2ced/dedba472-5e9c-489a-b80e-963af35f7eb6"
-          (reference "#PWR043") (unit 1)
+          (reference "#PWR046") (unit 1)
         )
       )
@@
   (symbol (lib_id "Device:C") (at 190.5 78.74 180) (unit 1)
     (in_bom yes) (on_board yes) (dnp no) (fields_autoplaced)
-    (property "Reference" "C28" (at 194.31 78.105 0)
+    (property "Reference" "C31" (at 194.31 78.105 0)
       (effects (font (size 1.27 1.27)) (justify right))
     )
@@
       (project "electrium-esc-v2"
         (path "/be00c12c-11fa-42cb-8a0b-46fcd24b2ced/dedba472-5e9c-489a-b80e-963af35f7eb6"
-          (reference "C28") (unit 1)
+          (reference "C31") (unit 1)
         )
       )
@@
   (symbol (lib_id "Device:C") (at 107.95 81.28 0) (unit 1)
     (in_bom yes) (on_board yes) (dnp no) (fields_autoplaced)
-    (property "Reference" "C25" (at 111.76 80.645 0)
+    (property "Reference" "C32" (at 111.76 80.645 0)
       (effects (font (size 1.27 1.27)) (justify left))
     )
@@
       (project "electrium-esc-v2"
         (path "/be00c12c-11fa-42cb-8a0b-46fcd24b2ced/dedba472-5e9c-489a-b80e-963af35f7eb6"
-          (reference "C25") (unit 1)
+          (reference "C32") (unit 1)
         )
       )
@@
   (symbol (lib_id "Device:R") (at 201.93 91.44 0) (unit 1)
     (in_bom yes) (on_board yes) (dnp no) (fields_autoplaced)
-    (property "Reference" "R19" (at 204.47 90.805 0)
+    (property "Reference" "R15" (at 204.47 90.805 0)
       (effects (font (size 1.27 1.27)) (justify left))
     )
@@
       (project "electrium-esc-v2"
         (path "/be00c12c-11fa-42cb-8a0b-46fcd24b2ced/dedba472-5e9c-489a-b80e-963af35f7eb6"
-          (reference "R19") (unit 1)
-        )
-      )
+          (reference "R15") (unit 1)
+        )
+      )
