File: MOSFETs.kicad_sch (KiCad schematic)
At the start: 0 parts

Commit message: changed pins
Parts:
- added C28: 3300u, Capacitor_THT:CP_Radial_D22.0mm_P10.00mm_SnapIn, symbol Device:C_Polarized_US
- added C29, C30, C31: 22u, Capacitor_SMD:CP_Elec_6.3x7.7, symbol Device:C
- added Q1, Q2, Q3, Q4, Q5, Q6: IRF3205, Package_TO_SOT_THT:TO-220-3_Vertical, symbol Transistor_FET:IRF3205
- added R17, R18, R19: .01, Resistor_SMD:R_2512_6332Metric_Pad1.40x3.35mm_HandSolder, symbol Device:R
Connections:
- new net GND: C28.2, C29.2, C30.2, C31.2, R17.2, R18.2, R19.2
- new net M_H2: Q4.1 (G)
- new net M_H3: Q5.1 (G)
- new net M_L2: Q3.1 (G)
- new net M_L3: Q6.1 (G)
- new net PWR_SRC: C28.1, C29.1, C30.1, C31.1, Q1.2 (D), Q3.2 (D), Q5.2 (D)
- new net SH1: Q1.3 (S), Q2.2 (D)
- new net SH2: Q3.3 (S), Q4.2 (D)
- new net SH3: Q5.3 (S), Q6.2 (D)
- new net SP1: Q2.3 (S), R17.1
- new net SP2: Q4.3 (S), R18.1
- new net SP3: Q6.3 (S), R19.1

Commit message: added nets to high level circuit
Changed lines of the file:
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@@
     (stroke (width 0) (type default))
-  )
-  (global_label "PWR_SRC" (shape input) (at 83.82 44.45 180) (fields_autoplaced)
-    (effects (font (size 1.27 1.27)) (justify right))
-    (property "Intersheetrefs" "${INTERSHEET_REFS}" (at 72.2057 44.45 0)
-      (effects (font (size 1.27 1.27)) (justify right) hide)
-    )
-  )
-  (global_label "PWR_SRC" (shape input) (at 86.36 66.04 180) (fields_autoplaced)
-    (effects (font (size 1.27 1.27)) (justify right))
-    (property "Intersheetrefs" "${INTERSHEET_REFS}" (at 74.7457 66.04 0)
-      (effects (font (size 1.27 1.27)) (justify right) hide)
-    )
   )
   (hierarchical_label "SP2" (shape input) (at 123.19 99.06 180) (fields_autoplaced)
@@
     (effects (font (size 1.27 1.27)) (justify right))
   )
+  (hierarchical_label "PWR_SRC" (shape input) (at 86.36 66.04 180) (fields_autoplaced)
+    (effects (font (size 1.27 1.27)) (justify right))
+  )
   (hierarchical_label "M_L2" (shape input) (at 115.57 73.66 180) (fields_autoplaced)
     (effects (font (size 1.27 1.27)) (justify right))
@@
     (effects (font (size 1.27 1.27)) (justify right))
   )
+  (hierarchical_label "PWR_SRC" (shape input) (at 83.82 44.45 180) (fields_autoplaced)
+    (effects (font (size 1.27 1.27)) (justify right))
+  )
