File: CAN.kicad_sch (KiCad schematic)
At the start: 2 parts

Commit message: changed pins
Parts:
- C25: renamed from C30; footprint Capacitor_SMD:C_0603_1608Metric -> (none)
- gave numbers to parts that had none: 1
Changed lines of the file:
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@@
   (symbol (lib_id "Interface_CAN_LIN:SN65HVD233") (at 143.51 93.98 0) (unit 1)
     (in_bom yes) (on_board yes) (dnp no) (fields_autoplaced)
-    (property "Reference" "U?" (at 145.4659 85.09 0)
+    (property "Reference" "U1" (at 145.4659 85.09 0)
       (effects (font (size 1.27 1.27)) (justify left))
     )
@@
       (project "CAN"
         (path "/02b8491d-2d12-4025-9131-d09e9a95b074"
-          (reference "U?") (unit 1)
+          (reference "U1") (unit 1)
         )
       )
@@
   (symbol (lib_id "power:GND") (at 143.51 107.95 0) (unit 1)
     (in_bom yes) (on_board yes) (dnp no) (fields_autoplaced)
-    (property "Reference" "#PWR?" (at 143.51 114.3 0)
+    (property "Reference" "#PWR02" (at 143.51 114.3 0)
       (effects (font (size 1.27 1.27)) hide)
     )
@@
       (project "CAN"
         (path "/02b8491d-2d12-4025-9131-d09e9a95b074"
-          (reference "#PWR?") (unit 1)
+          (reference "#PWR02") (unit 1)
         )
       )
       (project "electrium-esc-v2"
         (path "/be00c12c-11fa-42cb-8a0b-46fcd24b2ced/5d5f53ac-6241-4ef8-8b88-68f3e6833293"
-          (reference "#PWR042") (unit 1)
+          (reference "#PWR037") (unit 1)
         )
       )
@@
   (symbol (lib_id "Device:C") (at 168.91 95.25 0) (unit 1)
     (in_bom yes) (on_board yes) (dnp no) (fields_autoplaced)
-    (property "Reference" "C30" (at 172.72 94.615 0)
+    (property "Reference" "C25" (at 172.72 94.615 0)
       (effects (font (size 1.27 1.27)) (justify left))
     )
@@
       (effects (font (size 1.27 1.27)) (justify left))
     )
-    (property "Footprint" "Capacitor_SMD:C_0603_1608Metric" (at 169.8752 99.06 0)
+    (property "Footprint" "" (at 169.8752 99.06 0)
       (effects (font (size 1.27 1.27)) hide)
     )
@@
       (project "electrium-esc-v2"
         (path "/be00c12c-11fa-42cb-8a0b-46fcd24b2ced/5d5f53ac-6241-4ef8-8b88-68f3e6833293"
-          (reference "C30") (unit 1)
+          (reference "C25") (unit 1)
         )
       )
@@
   (symbol (lib_id "power:+3.3V") (at 143.51 77.47 0) (unit 1)
     (in_bom yes) (on_board yes) (dnp no) (fields_autoplaced)
-    (property "Reference" "#PWR?" (at 143.51 81.28 0)
+    (property "Reference" "#PWR01" (at 143.51 81.28 0)
       (effects (font (size 1.27 1.27)) hide)
     )
@@
       (project "CAN"
         (path "/02b8491d-2d12-4025-9131-d09e9a95b074"
-          (reference "#PWR?") (unit 1)
+          (reference "#PWR01") (unit 1)
         )
       )
       (project "electrium-esc-v2"
         (path "/be00c12c-11fa-42cb-8a0b-46fcd24b2ced/5d5f53ac-6241-4ef8-8b88-68f3e6833293"
-          (reference "#PWR041") (unit 1)
+          (reference "#PWR029") (unit 1)
         )
       )

Commit message: Re-annotate all components
Parts:
- renumbered C25 to C35, U1 to U?
Changed lines of the file:
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@@
   (symbol (lib_id "Interface_CAN_LIN:SN65HVD233") (at 143.51 93.98 0) (unit 1)
     (in_bom yes) (on_board yes) (dnp no) (fields_autoplaced)
-    (property "Reference" "U1" (at 145.4659 85.09 0)
+    (property "Reference" "U?" (at 145.4659 85.09 0)
       (effects (font (size 1.27 1.27)) (justify left))
     )
@@
       (project "CAN"
         (path "/02b8491d-2d12-4025-9131-d09e9a95b074"
-          (reference "U1") (unit 1)
+          (reference "U?") (unit 1)
         )
       )
@@
   (symbol (lib_id "power:GND") (at 143.51 107.95 0) (unit 1)
     (in_bom yes) (on_board yes) (dnp no) (fields_autoplaced)
-    (property "Reference" "#PWR02" (at 143.51 114.3 0)
+    (property "Reference" "#PWR?" (at 143.51 114.3 0)
       (effects (font (size 1.27 1.27)) hide)
     )
@@
       (project "CAN"
         (path "/02b8491d-2d12-4025-9131-d09e9a95b074"
-          (reference "#PWR02") (unit 1)
+          (reference "#PWR?") (unit 1)
         )
       )
       (project "electrium-esc-v2"
         (path "/be00c12c-11fa-42cb-8a0b-46fcd24b2ced/5d5f53ac-6241-4ef8-8b88-68f3e6833293"
-          (reference "#PWR037") (unit 1)
+          (reference "#PWR054") (unit 1)
         )
       )
@@
   (symbol (lib_id "Device:C") (at 168.91 95.25 0) (unit 1)
     (in_bom yes) (on_board yes) (dnp no) (fields_autoplaced)
-    (property "Reference" "C25" (at 172.72 94.615 0)
+    (property "Reference" "C35" (at 172.72 94.615 0)
       (effects (font (size 1.27 1.27)) (justify left))
     )
@@
       (project "electrium-esc-v2"
         (path "/be00c12c-11fa-42cb-8a0b-46fcd24b2ced/5d5f53ac-6241-4ef8-8b88-68f3e6833293"
-          (reference "C25") (unit 1)
+          (reference "C35") (unit 1)
         )
       )
@@
   (symbol (lib_id "power:+3.3V") (at 143.51 77.47 0) (unit 1)
     (in_bom yes) (on_board yes) (dnp no) (fields_autoplaced)
-    (property "Reference" "#PWR01" (at 143.51 81.28 0)
+    (property "Reference" "#PWR?" (at 143.51 81.28 0)
       (effects (font (size 1.27 1.27)) hide)
     )
@@
       (project "CAN"
         (path "/02b8491d-2d12-4025-9131-d09e9a95b074"
-          (reference "#PWR01") (unit 1)
+          (reference "#PWR?") (unit 1)
         )
       )
       (project "electrium-esc-v2"
         (path "/be00c12c-11fa-42cb-8a0b-46fcd24b2ced/5d5f53ac-6241-4ef8-8b88-68f3e6833293"
-          (reference "#PWR029") (unit 1)
+          (reference "#PWR053") (unit 1)
         )
       )

Commit message: Add proper footprints
Parts:
- C35: footprint (none) -> Capacitor_SMD:C_0603_1608Metric
Changed lines of the file:
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@@
       (effects (font (size 1.27 1.27)) (justify left))
     )
-    (property "Footprint" "" (at 169.8752 99.06 0)
+    (property "Footprint" "Capacitor_SMD:C_0603_1608Metric" (at 169.8752 99.06 0)
       (effects (font (size 1.27 1.27)) hide)
     )
