File: electrium-esc-v2.kicad_pcb (KiCad board)
At the start: 2 copper layers, 42.3 x 45.4 mm, 65 parts, among them IC1 LMR36510FADDAR, J1 CAN, J2 Conn_01x02, J3 USB_B_Micro, J4 Debugger Pins, J5 GPIO, U1 W25Q128JVS, U2 NCP1117-3.3_SOT223, U3 RP2040, U4 DRV8323HRTAR, U5 NRF24L01_Breakout, U6 SN65HVD233, Y1 ABLS-12.000MHZ-B4-T

Commit message: pcb designed
Parts:
- removed C28: 4.3p, Capacitor_SMD:C_0603_1608Metric
- removed C29: 47u, Capacitor_SMD:C_0603_1608Metric
- removed R16: 47k, Resistor_SMD:R_0603_1608Metric
- removed R17, R18: 100k, Resistor_SMD:R_0603_1608Metric
- removed R19: 43.2k, Resistor_SMD:R_0603_1608Metric
- added C31: 4.3p, Capacitor_SMD:C_0603_1608Metric, F.Cu at (190.9, 80.8)
- added C32: 4.7u, Capacitor_SMD:C_0603_1608Metric, F.Cu at (204.6, 82.2)
- added C33: 220n, Capacitor_SMD:C_0603_1608Metric, F.Cu at (206.2, 82.2)
- added C34: 47u, Capacitor_SMD:C_0603_1608Metric, F.Cu at (189.3, 80.8)
- added C35: 0.1u, Capacitor_SMD:C_0603_1608Metric, F.Cu at (178.4, 89.0)
- added J6: Conn_01x03_Pin, Connector_PinHeader_2.54mm:PinHeader_1x03_P2.54mm_Vertical, F.Cu at (186.5, 77.0)
- added Q1: IRF3205, Package_TO_SOT_THT:TO-220-3_Vertical, F.Cu at (239.8, 112.7)
- added Q2: IRF3205, Package_TO_SOT_THT:TO-220-3_Vertical, F.Cu at (240.0, 98.5)
- added Q3: IRF3205, Package_TO_SOT_THT:TO-220-3_Vertical, F.Cu at (239.8, 85.5)
- added Q4: IRF3205, Package_TO_SOT_THT:TO-220-3_Vertical, F.Cu at (245.0, 107.7)
- added Q5: IRF3205, Package_TO_SOT_THT:TO-220-3_Vertical, F.Cu at (245.0, 93.5)
- added Q6: IRF3205, Package_TO_SOT_THT:TO-220-3_Vertical, F.Cu at (245.0, 80.5)
- added TP1: FaultTest, TestPoint:TestPoint_Pad_D2.5mm, B.Cu at (214.8, 91.0)
- added VR1: VG039NCHXTB204, VG039NCHXTB204:VG039NCHXTB204, F.Cu at (192.0, 113.8)
- added VR2: VG039NCHXTB204, VG039NCHXTB204:VG039NCHXTB204, F.Cu at (203.6, 113.8)
- added VR3: VG039NCHXTB204, VG039NCHXTB204:VG039NCHXTB204, F.Cu at (197.8, 113.8)
- added VR4: VG039NCHXTB204, VG039NCHXTB204:VG039NCHXTB204, F.Cu at (217.0, 78.8)
- C1, C2: value 27p -> 100n
- C10: value 1u -> 10u; moved to F.Cu
- C11, C12: value 100n -> 10u; moved to F.Cu
- C13, C14: value 100n -> 1u; moved to F.Cu
- C15, C6, C7, C9: moved to F.Cu
- C16: value 100n -> 27p; moved to F.Cu
- C17: value 10u -> 27p; footprint Capacitor_THT:CP_Radial_D5.0mm_P2.00mm -> Capacitor_SMD:C_0603_1608Metric
- C18: value 0.1u -> 1u
- C19: value 47u -> 47n; footprint Capacitor_THT:CP_Radial_D5.0mm_P2.00mm -> Capacitor_SMD:C_0603_1608Metric
- C21: value 47n -> 0.1u
- C22: value 1u -> 47u; footprint Capacitor_SMD:C_0603_1608Metric -> Capacitor_THT:CP_Radial_D4.0mm_P1.50mm
- C24: value 47u -> 22u; footprint Capacitor_THT:CP_Radial_D5.0mm_P2.00mm -> Capacitor_SMD:CP_Elec_6.3x7.7
- C25: value 4.7u -> 22u; footprint Capacitor_SMD:C_0603_1608Metric -> Capacitor_SMD:CP_Elec_6.3x7.7
- C26: value 220n -> 22u; footprint Capacitor_SMD:C_0603_1608Metric -> Capacitor_SMD:CP_Elec_6.3x7.7
- C27: value 100n -> 3300u; footprint Capacitor_SMD:C_0603_1608Metric -> Capacitor_THT:CP_Radial_D22.0mm_P10.00mm_SnapIn; moved to B.Cu
- C3: value 10u -> 100n
- C30: value 0.1u -> 100n; moved to F.Cu
- C5: value 10u -> 100n; moved to F.Cu
- C8: value 1u -> 100n; moved to F.Cu
- J2: value Conn_01x02 -> USB_B_Micro; footprint Connector_PinHeader_2.54mm:PinHeader_1x02_P2.54mm_Vertical -> Connector_USB:USB_Micro-B_Molex-105017-0001
- J3: value USB_B_Micro -> GPIO; footprint Connector_USB:USB_Micro-B_Molex-105017-0001 -> Connector_PinSocket_2.54mm:PinSocket_1x07_P2.54mm_Vertical
- J4: value Debugger Pins -> Conn_01x02; footprint Connector_JST:JST_XH_B4B-XH-A_1x04_P2.50mm_Vertical -> Connector_PinHeader_2.54mm:PinHeader_1x02_P2.54mm_Vertical
- J5: value GPIO -> Debugger Pins; footprint Connector_PinSocket_2.54mm:PinSocket_1x07_P2.54mm_Vertical -> Connector_JST:JST_XH_B4B-XH-A_1x04_P2.50mm_Vertical
- R10: value 10k -> .01; footprint Resistor_SMD:R_0603_1608Metric -> Resistor_SMD:R_2512_6332Metric_Pad1.40x3.35mm_HandSolder; moved to B.Cu
- R11, R12: value 75k -> .01; footprint Resistor_SMD:R_0603_1608Metric -> Resistor_SMD:R_2512_6332Metric_Pad1.40x3.35mm_HandSolder; moved to B.Cu
- R13: value 10k -> 100k
- R14: value 75k -> 100k
- R15: value 47k -> 43.2k
- R3: value 1k -> 27; moved to F.Cu
- R4: value DNF -> 27
- R5: value 1k -> DNF
- R6, R7: value 27 -> 1k
- U1: value W25Q128JVS -> NCP1117-3.3_SOT223; footprint Package_SO:SOIC-8_5.23x5.23mm_P1.27mm -> Package_TO_SOT_SMD:SOT-223-3_TabPin2
- U2: value NCP1117-3.3_SOT223 -> W25Q128JVS; footprint Package_TO_SOT_SMD:SOT-223-3_TabPin2 -> Package_SO:SOIC-8_5.23x5.23mm_P1.27mm
- U3: footprint ext_footprint:RP2040-QFN-56 -> Footprints:RP2040-QFN-56
- Y1: footprint ext_footprint:Crystal_SMD_HC49-US -> Footprints:Crystal_SMD_HC49-US
- moved C24 80.6 mm to (226.0, 79.0), turned to 180 degrees
- moved J5 68.4 mm to (178.0, 114.0), turned to 90 degrees
- moved C26 65.6 mm to (225.9, 108.2)
- moved R12 64.3 mm to (226.8, 87.6), turned to 180 degrees
- moved R10 63.3 mm to (226.9, 115.2), turned to 180 degrees
- moved R11 61.9 mm to (227.0, 100.8), turned to 180 degrees
- moved C21 61.6 mm to (219.6, 108.2), turned to 0 degrees
- moved C2 60.4 mm to (209.0, 110.2), turned to -90 degrees
- moved D2 60.2 mm to (193.4, 105.8), turned to 0 degrees
- moved R2 60.1 mm to (196.2, 105.6), turned to 0 degrees
- moved C22 59.6 mm to (217.8, 85.0), turned to -90 degrees
- moved C25 58.5 mm to (226.0, 93.0)
- moved C20 58.0 mm to (217.2, 107.2), turned to 90 degrees
- moved C27 58.0 mm to (219.2, 114.8), turned to 180 degrees
- moved C9 56.2 mm to (214.0, 105.6), turned to -90 degrees
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Connections:
- net /MCU (RP2040)/ENABLE renamed /MCU/ENABLE
- net /MCU (RP2040)/OUT_H1 renamed /MCU/OUT_H1
- net /MCU (RP2040)/OUT_H2 renamed /MCU/OUT_H2
- net /MCU (RP2040)/OUT_H3 renamed /MCU/OUT_H3
- net /MCU (RP2040)/OUT_L1 renamed /MCU/OUT_L1
- net /MCU (RP2040)/OUT_L2 renamed /MCU/OUT_L2
- net /MCU (RP2040)/OUT_L3 renamed /MCU/OUT_L3
- net /MCU (RP2040)/SENS1 renamed /MCU/SENS1
- net /MCU (RP2040)/SENS2 renamed /MCU/SENS2
- net /MCU (RP2040)/SENS3 renamed /MCU/SENS3
- C1 pad 1: /MCU (RP2040)/XIN -> +1V1
- C11 pad 1: +3.3V -> VBUS
- C12 pad 1: +3.3V -> Net-(J6-Pin_3)
- C13 pad 1: +3.3V -> +1V1
- C16 pad 1: +3.3V -> /MCU/XIN
- C17 pad 1: +3.3V -> Net-(C17-Pad1)
- C18 pad 1: PWR_SRC -> Net-(U4-DVDD)
- C19 pad 1: PWR_SRC -> Net-(U4-CPL)
- C19 pad 2: GND -> Net-(U4-CPH)
- C2 pad 1: Net-(C2-Pad1) -> +1V1
- C21 pad 1: Net-(U4-CPL) -> PWR_SRC
- C21 pad 2: Net-(U4-CPH) -> GND
- C22 pad 1: Net-(U4-DVDD) -> PWR_SRC
- C24 pad 1: +3.3V -> PWR_SRC
- C27 pad 1: Net-(IC1-BOOT) -> PWR_SRC
- C27 pad 2: Net-(IC1-SW) -> GND
- C3 pad 1: VBUS -> +3.3V
- C30 pad 1: +3.3V -> Net-(IC1-BOOT)
- C30 pad 2: GND -> Net-(IC1-SW)
- C6 pad 1: +1V1 -> +3.3V
- C7 pad 1: +1V1 -> +3.3V
- C8 pad 1: +1V1 -> +3.3V
- IC1 pad 5: /Buck Converter (LMR36510FADDAR)/FB -> Net-(IC1-FB)
- J1 pad 2: /CAN/CANL -> /CAN/CAN-
- J1 pad 3: /CAN/CANH -> /CAN/CAN+
- J2 pad 1: /MCU (RP2040)/~{USB_BOOT} -> VBUS
- J2 pad 2: GND -> /MCU/USB_D-
- J3 pad 1: VBUS -> Net-(J3-Pin_1)
- J3 pad 2: /MCU (RP2040)/USB_D- -> Net-(J3-Pin_2)
- J3 pad 3: /MCU (RP2040)/USB_D+ -> Net-(J3-Pin_3)
- J3 pad 4: unconnected-(J3-ID-Pad4) -> Net-(J3-Pin_4)
- J3 pad 5: GND -> Net-(J3-Pin_5)
- J3 pad 6: GND -> Net-(J3-Pin_6)
- J4 pad 1: +3.3V -> /MCU/~{USB_BOOT}
- J4 pad 2: /MCU (RP2040)/SWCLK -> GND
- J5 pad 1: Net-(J5-Pin_1) -> +3.3V
- J5 pad 2: Net-(J5-Pin_2) -> /MCU/SWCLK
- J5 pad 3: Net-(J5-Pin_3) -> GND
- J5 pad 4: Net-(J5-Pin_4) -> /MCU/SWD
- L1 pad 2: +3.3V -> LMR_3v3
- R10 pad 1: /MCU (RP2040)/MODE -> /MOSFETs/SP1
- R11 pad 1: +3.3V -> /MOSFETs/SP2
- R11 pad 2: /MCU (RP2040)/IDRIVE -> GND
- R12 pad 1: /MCU (RP2040)/IDRIVE -> /MOSFETs/SP3
- R13 pad 1: +3.3V -> Net-(IC1-PG)
- R13 pad 2: Net-(U4-VDS) -> LMR_3v3
- R14 pad 1: Net-(U4-VDS) -> LMR_3v3
- R14 pad 2: GND -> Net-(IC1-FB)
- R15 pad 1: +3.3V -> Net-(IC1-FB)
- R15 pad 2: Net-(U4-GAIN) -> GND
- R2 pad 2: (no net) -> /MCU/LED
- R3 pad 1: /MCU (RP2040)/QSPI_SS -> /MCU/USB_D+
- R3 pad 2: /MCU (RP2040)/~{USB_BOOT} -> /MCU/USB_DP
- R4 pad 1: +3.3V -> /MCU/USB_D-
- R4 pad 2: /MCU (RP2040)/QSPI_SS -> /MCU/USB_DN
- R5 pad 1: /MCU (RP2040)/XOUT -> +3.3V
- R5 pad 2: Net-(C2-Pad1) -> /MCU/QSPI_SS
- R6 pad 1: /MCU (RP2040)/USB_D+ -> /MCU/QSPI_SS
- R6 pad 2: Net-(U3-USB_DP) -> /MCU/~{USB_BOOT}
- R7 pad 1: /MCU (RP2040)/USB_D- -> /MCU/XOUT
- R7 pad 2: Net-(U3-USB_DM) -> Net-(C17-Pad1)
- R9 pad 1: /MCU (RP2040)/NFAULT -> +3.3V
- R9 pad 2: +3.3V -> /MCU/NFAULT
- U1 pad 1: /MCU (RP2040)/QSPI_SS -> GND
- U1 pad 2: /MCU (RP2040)/QSPI_SD1 -> Net-(J6-Pin_3)
- U1 pad 3: /MCU (RP2040)/QSPI_SD2 -> VBUS
- U2 pad 1: GND -> /MCU/QSPI_SS
- U2 pad 2: +3.3V -> /MCU/QSPI_SD1
- U2 pad 3: VBUS -> /MCU/QSPI_SD2
- U3 pad 11: Net-(J5-Pin_4) -> Net-(J3-Pin_4)
- U3 pad 12: Net-(J5-Pin_5) -> Net-(J3-Pin_5)
- U3 pad 13: Net-(J5-Pin_6) -> Net-(J3-Pin_6)
- U3 pad 14: Net-(J5-Pin_7) -> Net-(J3-Pin_7)
- U3 pad 15: /MCU (RP2040)/CANTX -> /MCU/CANTX
- U3 pad 16: /MCU (RP2040)/CANRX -> /MCU/CANRX
- U3 pad 17: /MCU (RP2040)/LBK -> /MCU/LBK
- U3 pad 18: /MCU (RP2040)/LED -> /MCU/LED
- U3 pad 2: /MCU (RP2040)/NRF_MISO -> /MCU/NRF_MISO
- U3 pad 20: /MCU (RP2040)/XIN -> /MCU/XIN
- U3 pad 21: /MCU (RP2040)/XOUT -> /MCU/XOUT
- U3 pad 24: /MCU (RP2040)/SWCLK -> /MCU/SWCLK
- U3 pad 25: /MCU (RP2040)/SWD -> /MCU/SWD
- U3 pad 3: /MCU (RP2040)/NRF_CS -> /MCU/NRF_CSN
- U3 pad 35: /MCU (RP2040)/IDRIVE -> unconnected-(U3-GPIO23-Pad35)
- U3 pad 36: /MCU (RP2040)/MODE -> unconnected-(U3-GPIO24-Pad36)
- U3 pad 37: /MCU (RP2040)/NFAULT -> /MCU/NFAULT
- U3 pad 4: /MCU (RP2040)/NRF_CLK -> /MCU/NRF_SCLK
- U3 pad 46: Net-(U3-USB_DM) -> /MCU/USB_DN
- U3 pad 47: Net-(U3-USB_DP) -> /MCU/USB_DP
- U3 pad 5: /MCU (RP2040)/NRF_MOSI -> /MCU/NRF_MOSI
- U3 pad 51: /MCU (RP2040)/QSPI_SD3 -> /MCU/QSPI_SD3
- U3 pad 52: /MCU (RP2040)/QSPI_SCLK -> /MCU/QSPI_SCLK
- U3 pad 53: /MCU (RP2040)/QSPI_SD0 -> /MCU/QSPI_SD0
- U3 pad 54: /MCU (RP2040)/QSPI_SD2 -> /MCU/QSPI_SD2
- U3 pad 55: /MCU (RP2040)/QSPI_SD1 -> /MCU/QSPI_SD1
- U3 pad 56: /MCU (RP2040)/QSPI_SS -> /MCU/QSPI_SS
- U3 pad 6: /MCU (RP2040)/NRF_CE -> /MCU/NRF_CE
- U3 pad 7: Net-(J5-Pin_1) -> Net-(J3-Pin_1)
- U3 pad 8: Net-(J5-Pin_2) -> Net-(J3-Pin_2)
- U3 pad 9: Net-(J5-Pin_3) -> Net-(J3-Pin_3)
- U4 pad 10: /Motor Driver (DRV8323)/SN1 -> GND
- U4 pad 11: /Motor Driver (DRV8323)/SN2 -> GND
- U4 pad 12: /Motor Driver (DRV8323)/SP2 -> /MOSFETs/SP2
- U4 pad 13: /Motor Driver (DRV8323)/M_L2 -> /MOSFETs/M_L2
- U4 pad 14: /Motor Driver (DRV8323)/SH2 -> /MOSFETs/SH2
- U4 pad 15: /Motor Driver (DRV8323)/M_H2 -> /MOSFETs/M_H2
- U4 pad 16: /Motor Driver (DRV8323)/M_H3 -> /MOSFETs/M_H3
- U4 pad 17: /Motor Driver (DRV8323)/SH3 -> /MOSFETs/SH3
- U4 pad 18: /Motor Driver (DRV8323)/M_L3 -> /MOSFETs/M_L3
- U4 pad 19: /Motor Driver (DRV8323)/SP3 -> /MOSFETs/SP3
- U4 pad 20: /Motor Driver (DRV8323)/SN3 -> GND
- U4 pad 25: /MCU (RP2040)/NFAULT -> /MCU/NFAULT
- U4 pad 26: /MCU (RP2040)/MODE -> MODE
- U4 pad 27: /MCU (RP2040)/IDRIVE -> IDRIVE
- U4 pad 28: Net-(U4-VDS) -> VDS
- U4 pad 29: Net-(U4-GAIN) -> GAIN
- U4 pad 6: /Motor Driver (DRV8323)/M_H1 -> /MOSFETs/M_H1
- U4 pad 7: /Motor Driver (DRV8323)/SH1 -> /MOSFETs/SH1
- U4 pad 8: /Motor Driver (DRV8323)/M_L1 -> /MOSFETs/M_L1
- U4 pad 9: /Motor Driver (DRV8323)/SP1 -> /MOSFETs/SP1
- U5 pad 3: (no net) -> /MCU/NRF_CE
- U5 pad 4: (no net) -> /MCU/NRF_CSN
- U5 pad 5: (no net) -> /MCU/NRF_SCLK
- U5 pad 6: (no net) -> /MCU/NRF_MOSI
- U5 pad 7: (no net) -> /MCU/NRF_MISO
- U6 pad 1: (no net) -> /MCU/CANTX
- U6 pad 4: (no net) -> /MCU/CANRX
- U6 pad 5: (no net) -> /MCU/LBK
- U6 pad 6: /CAN/CANL -> /CAN/CAN+
- U6 pad 7: /CAN/CANH -> /CAN/CAN-
- Y1 pad 1: /MCU (RP2040)/XIN -> /MCU/XIN
- Y1 pad 2: Net-(C2-Pad1) -> Net-(C17-Pad1)
Routing:
- net +3.3V: track 94.3 -> 263.1 mm, vias 11 -> 15
- net PWR_SRC: track 0.07 -> 56.9 mm, vias 0 -> 1
- net Net-(J3-Pin_7): track 0.00 -> 55.8 mm, vias 0 -> 3
- net Net-(J3-Pin_6): track 0.00 -> 51.1 mm, vias 0 -> 1
- net Net-(J3-Pin_5): track 0.00 -> 48.4 mm, vias 0 -> 3
- net Net-(J3-Pin_4): track 0.00 -> 44.6 mm, vias 0 -> 4
- net /MCU/SWD: track 0.00 -> 43.7 mm, vias 0 -> 1
- net /MCU/QSPI_SS: track 0.00 -> 42.7 mm, vias 0 -> 5
- net Net-(J3-Pin_3): track 0.00 -> 42.7 mm, vias 0 -> 2
- net /MOSFETs/M_L3: track 0.00 -> 42.3 mm, vias 0 -> 1
- net Net-(J3-Pin_2): track 0.00 -> 40.9 mm, vias 0 -> 2
- net Net-(J3-Pin_1): track 0.00 -> 40.5 mm, vias 0 -> 2
- net GAIN: track 0.00 -> 38.2 mm, vias 0 -> 2
- net /MCU/USB_DN: track 0.00 -> 37.6 mm, vias 0 -> 2
- net /MCU/USB_DP: track 0.00 -> 37.3 mm, vias 0 -> 2
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- added copper zone on B.Cu, net /MOSFETs/SH1
- added copper zone on F.Cu, net /MOSFETs/SH1
- added copper zone on B.Cu, net /MOSFETs/SH2
- added copper zone on F.Cu, net /MOSFETs/SH2
- added copper zone on B.Cu, net /MOSFETs/SH3
- added copper zone on F.Cu, net /MOSFETs/SH3
- added copper zone on B.Cu, net /MOSFETs/SP1
- added copper zone on F.Cu, net /MOSFETs/SP1
- added copper zone on B.Cu, net /MOSFETs/SP2
- added copper zone on F.Cu, net /MOSFETs/SP2
- added copper zone on B.Cu, net /MOSFETs/SP3
- added copper zone on F.Cu, net /MOSFETs/SP3
- added copper zone on B.Cu, net GND
- added copper zone on F.Cu, net GND
- removed copper zone on B.Cu, net +3.3V
- removed copper zone on F.Cu, net /Buck Converter (LMR36510FADDAR)/FB
Other:
- board size 42.3 x 45.4 mm -> 75.4 x 42 mm
