File: electrium-esc-v2.kicad_pcb (KiCad board)
At the start: 2 copper layers, 45 x 62 mm, 74 parts, among them IC1 LMR36510FADDAR, J1 CAN, J2 USB_B_Micro, J3 GPIO, J4 Conn_01x02, J5 Debugger Pins, J6 3.3VJumper, Q1 IRF3205, Q2 IRF3205, Q3 IRF3205, Q4 IRF3205, Q5 IRF3205, Q6 IRF3205, U1 NCP1117-3.3_SOT223, U2 W25Q128JVS, U3 RP2040, U4 DRV8323HRTAR, U5 NRF24L01_Breakout, U6 SN65HVD233, Y1 ABLS-12.000MHZ-B4-T

Commit message: Final PCB V2
Routing:
- net GND: track 94.9 -> 101.9 mm
- net /MOSFETs/M_H1: track 35.2 -> 34.1 mm
Changed lines of the file:
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@@
   (segment (start 175.4794 74.8438) (end 175.0568 74.8438) (width 0.1778) (layer "F.Cu") (net 1))
   (segment (start 194.2592 67.326) (end 194.2592 66.548) (width 0.2032) (layer "F.Cu") (net 1))
+  (segment (start 203.0476 51.9576) (end 203.0476 58.9576) (width 0.254) (layer "F.Cu") (net 1))
   (segment (start 179.712 65.34) (end 179.7509 65.3789) (width 0.1778) (layer "F.Cu") (net 1))
   (segment (start 173.1512 65.3796) (end 173.1512 65.3028) (width 0.2032) (layer "F.Cu") (net 1))
@@
   (segment (start 176.8348 52.9844) (end 176.8856 53.0352) (width 0.2032) (layer "F.Cu") (net 1))
   (via (at 181.4576 69.6468) (size 0.8) (drill 0.4) (layers "F.Cu" "B.Cu") (net 1))
-  (via (at 191.4128 98.0642) (size 0.5) (drill 0.3) (layers "F.Cu" "B.Cu") (free) (net 1))
+  (via (at 191.4144 97.3836) (size 0.5) (drill 0.3) (layers "F.Cu" "B.Cu") (free) (net 1))
   (via (at 195.7324 64.3128) (size 0.5) (drill 0.3) (layers "F.Cu" "B.Cu") (net 1))
   (via (at 181.4576 67.8688) (size 0.8) (drill 0.4) (layers "F.Cu" "B.Cu") (net 1))
@@
   (via (at 171.6532 60.3504) (size 0.8) (drill 0.4) (layers "F.Cu" "B.Cu") (free) (net 1))
   (via (at 167.7416 60.3504) (size 0.8) (drill 0.4) (layers "F.Cu" "B.Cu") (free) (net 1))
-  (via (at 190.8032 98.0642) (size 0.5) (drill 0.3) (layers "F.Cu" "B.Cu") (free) (net 1))
+  (via (at 190.8048 97.3836) (size 0.5) (drill 0.3) (layers "F.Cu" "B.Cu") (free) (net 1))
   (via (at 183.1848 67.818) (size 0.8) (drill 0.4) (layers "F.Cu" "B.Cu") (net 1))
-  (via (at 191.9716 98.0642) (size 0.5) (drill 0.3) (layers "F.Cu" "B.Cu") (free) (net 1))
+  (via (at 191.9732 97.3836) (size 0.5) (drill 0.3) (layers "F.Cu" "B.Cu") (free) (net 1))
   (via (at 170.9928 63.1444) (size 0.8) (drill 0.4) (layers "F.Cu" "B.Cu") (net 1))
   (via (at 182.3212 66.9544) (size 0.8) (drill 0.4) (layers "F.Cu" "B.Cu") (net 1))
-  (via (at 176.63 97.9932) (size 0.5) (drill 0.3) (layers "F.Cu" "B.Cu") (free) (net 1))
-  (via (at 163.068 99.1616) (size 0.5) (drill 0.3) (layers "F.Cu" "B.Cu") (free) (net 1))
+  (via (at 176.63 97.4852) (size 0.5) (drill 0.3) (layers "F.Cu" "B.Cu") (free) (net 1))
+  (via (at 163.068 97.6376) (size 0.5) (drill 0.3) (layers "F.Cu" "B.Cu") (free) (net 1))
   (via (at 192.3288 78.2828) (size 0.5) (drill 0.3) (layers "F.Cu" "B.Cu") (net 1))
   (via (at 180.594 68.7832) (size 0.8) (drill 0.4) (layers "F.Cu" "B.Cu") (net 1))
   (via (at 199.6948 79.7052) (size 0.5) (drill 0.3) (layers "F.Cu" "B.Cu") (net 1))
   (via (at 162.2552 93.3704) (size 0.8) (drill 0.4) (layers "F.Cu" "B.Cu") (free) (net 1))
-  (via (at 163.068 102.4128) (size 0.5) (drill 0.3) (layers "F.Cu" "B.Cu") (free) (net 1))
-  (via (at 177.1888 97.9932) (size 0.5) (drill 0.3) (layers "F.Cu" "B.Cu") (free) (net 1))
+  (via (at 163.068 102.8192) (size 0.5) (drill 0.3) (layers "F.Cu" "B.Cu") (free) (net 1))
+  (via (at 177.1888 97.4852) (size 0.5) (drill 0.3) (layers "F.Cu" "B.Cu") (free) (net 1))
   (via (at 172.0596 73.9648) (size 0.5) (drill 0.3) (layers "F.Cu" "B.Cu") (net 1))
   (via (at 194.818 65.9892) (size 0.5) (drill 0.3) (layers "F.Cu" "B.Cu") (net 1))
@@
   (via (at 160.5788 90.8304) (size 0.8) (drill 0.4) (layers "F.Cu" "B.Cu") (free) (net 1))
   (via (at 183.1848 68.7832) (size 0.8) (drill 0.4) (layers "F.Cu" "B.Cu") (net 1))
-  (via (at 161.8996 102.4128) (size 0.5) (drill 0.3) (layers "F.Cu" "B.Cu") (free) (net 1))
+  (via (at 161.8996 102.8192) (size 0.5) (drill 0.3) (layers "F.Cu" "B.Cu") (free) (net 1))
   (via (at 192.5812 101.3968) (size 0.5) (drill 0.3) (layers "F.Cu" "B.Cu") (free) (net 1))
   (via (at 203.0476 72.5424) (size 0.5) (drill 0.3) (layers "F.Cu" "B.Cu") (net 1))
@@
   (via (at 181.4576 68.7832) (size 0.8) (drill 0.4) (layers "F.Cu" "B.Cu") (net 1))
   (via (at 162.2552 89.5604) (size 0.8) (drill 0.4) (layers "F.Cu" "B.Cu") (free) (net 1))
-  (via (at 176.0204 97.9932) (size 0.5) (drill 0.3) (layers "F.Cu" "B.Cu") (free) (net 1))
-  (via (at 161.29 99.1616) (size 0.5) (drill 0.3) (layers "F.Cu" "B.Cu") (free) (net 1))
+  (via (at 176.0204 97.4852) (size 0.5) (drill 0.3) (layers "F.Cu" "B.Cu") (free) (net 1))
+  (via (at 161.29 97.6376) (size 0.5) (drill 0.3) (layers "F.Cu" "B.Cu") (free) (net 1))
   (via (at 199.136 51.816) (size 0.5) (drill 0.3) (layers "F.Cu" "B.Cu") (net 1))
   (via (at 167.8432 56.5912) (size 0.8) (drill 0.4) (layers "F.Cu" "B.Cu") (free) (net 1))
   (via (at 163.8808 93.3704) (size 0.8) (drill 0.4) (layers "F.Cu" "B.Cu") (free) (net 1))
-  (via (at 192.5812 98.0642) (size 0.5) (drill 0.3) (layers "F.Cu" "B.Cu") (free) (net 1))
-  (via (at 177.7984 97.9932) (size 0.5) (drill 0.3) (layers "F.Cu" "B.Cu") (free) (net 1))
+  (via (at 192.5828 97.3836) (size 0.5) (drill 0.3) (layers "F.Cu" "B.Cu") (free) (net 1))
+  (via (at 177.7984 97.4852) (size 0.5) (drill 0.3) (layers "F.Cu" "B.Cu") (free) (net 1))
   (via (at 175.1584 77.216) (size 0.5) (drill 0.3) (layers "F.Cu" "B.Cu") (net 1))
   (via (at 185.1152 78.994) (size 0.5) (drill 0.3) (layers "F.Cu" "B.Cu") (net 1))
@@
   (via (at 198.9836 54.1528) (size 0.5) (drill 0.3) (layers "F.Cu" "B.Cu") (net 1))
   (via (at 176.9364 53.0352) (size 0.5) (drill 0.3) (layers "F.Cu" "B.Cu") (net 1))
-  (via (at 161.29 102.4128) (size 0.5) (drill 0.3) (layers "F.Cu" "B.Cu") (free) (net 1))
+  (via (at 161.29 102.8192) (size 0.5) (drill 0.3) (layers "F.Cu" "B.Cu") (free) (net 1))
   (via (at 191.9716 101.3968) (size 0.5) (drill 0.3) (layers "F.Cu" "B.Cu") (free) (net 1))
   (via (at 198.755 62.992) (size 0.5) (drill 0.3) (layers "F.Cu" "B.Cu") (net 1))
@@
   (via (at 181.4576 66.9544) (size 0.8) (drill 0.4) (layers "F.Cu" "B.Cu") (net 1))
   (via (at 177.7984 101.5492) (size 0.5) (drill 0.3) (layers "F.Cu" "B.Cu") (free) (net 1))
-  (via (at 162.4584 102.4128) (size 0.5) (drill 0.3) (layers "F.Cu" "B.Cu") (free) (net 1))
+  (via (at 162.4584 102.8192) (size 0.5) (drill 0.3) (layers "F.Cu" "B.Cu") (free) (net 1))
   (via (at 180.594 67.8688) (size 0.8) (drill 0.4) (layers "F.Cu" "B.Cu") (net 1))
   (via (at 179.6796 55.9308) (size 0.5) (drill 0.3) (layers "F.Cu" "B.Cu") (net 1))
@@
   (via (at 182.3212 69.6468) (size 0.8) (drill 0.4) (layers "F.Cu" "B.Cu") (net 1))
   (via (at 191.4128 101.3968) (size 0.5) (drill 0.3) (layers "F.Cu" "B.Cu") (free) (net 1))
-  (via (at 161.8996 99.1616) (size 0.5) (drill 0.3) (layers "F.Cu" "B.Cu") (free) (net 1))
+  (via (at 161.8996 97.6376) (size 0.5) (drill 0.3) (layers "F.Cu" "B.Cu") (free) (net 1))
   (via (at 162.2552 88.2904) (size 0.8) (drill 0.4) (layers "F.Cu" "B.Cu") (free) (net 1))
   (via (at 199.6948 78.8924) (size 0.5) (drill 0.3) (layers "F.Cu" "B.Cu") (net 1))
   (via (at 163.8808 92.1004) (size 0.8) (drill 0.4) (layers "F.Cu" "B.Cu") (free) (net 1))
-  (via (at 162.4584 99.1616) (size 0.5) (drill 0.3) (layers "F.Cu" "B.Cu") (free) (net 1))
+  (via (at 162.4584 97.6376) (size 0.5) (drill 0.3) (layers "F.Cu" "B.Cu") (free) (net 1))
   (via (at 203.4032 66.6496) (size 0.8) (drill 0.4) (layers "F.Cu" "B.Cu") (net 1))
   (via (at 189.5348 72.6948) (size 0.8) (drill 0.4) (layers "F.Cu" "B.Cu") (net 1))
@@
   (segment (start 176.784 82.3564) (end 176.784 83.5152) (width 0.254) (layer "F.Cu") (net 77))
   (via (at 176.784 83.5152) (size 0.5) (drill 0.3) (layers "F.Cu" "B.Cu") (net 77))
-  (segment (start 174.9366 83.5152) (end 167.2844 91.1674) (width 0.254) (layer "B.Cu") (net 77))
-  (segment (start 167.2844 91.1674) (end 167.2844 95.8088) (width 0.254) (layer "B.Cu") (net 77))
-  (segment (start 176.784 83.5152) (end 174.9366 83.5152) (width 0.254) (layer "B.Cu") (net 77))
+  (segment (start 176.784 83.5152) (end 167.2844 93.0148) (width 0.254) (layer "B.Cu") (net 77))
+  (segment (start 167.2844 93.0148) (end 167.2844 95.8088) (width 0.254) (layer "B.Cu") (net 77))
   (segment (start 178.1556 82.277652) (end 178.1556 82.9564) (width 0.254) (layer "F.Cu") (net 78))
   (segment (start 178.115948 69.54) (end 177.781 69.874947) (width 0.254) (layer "F.Cu") (net 78))
@@
     (polygon
       (pts
-        (xy 160.8836 98.8568)
-        (xy 163.5252 98.8568)
-        (xy 163.5252 102.8192)
-        (xy 160.8836 102.8192)
+        (xy 160.8836 97.3328)
+        (xy 163.5252 97.3328)
+        (xy 163.5252 103.2764)
+        (xy 160.8836 103.2764)
       )
     )
@@
     (polygon
       (pts
-        (xy 190.3968 97.7086)
-        (xy 193.0384 97.7086)
-        (xy 193.0384 101.7726)
-        (xy 190.3968 101.7726)
+        (xy 190.3968 97.1296)
+        (xy 193.0384 97.1296)
+        (xy 193.0384 101.7524)
+        (xy 190.3968 101.7524)
       )
     )
@@
     (polygon
       (pts
-        (xy 175.614 97.7594)
-        (xy 178.2556 97.7594)
+        (xy 175.614 97.1498)
+        (xy 178.2556 97.1498)
         (xy 178.2556 101.9758)
         (xy 175.614 101.9758)
@@
         (xy 197.5104 100.305603)
         (xy 189.7888 100.305603)
-        (xy 189.7888 98.832403)
-        (xy 194.099791 98.832403)
+        (xy 189.7888 98.476803)
+        (xy 194.099791 98.476803)
         (xy 194.099791 98.044)
       )
@@
       (pts
         (xy 182.937809 97.918003)
-        (xy 182.937809 100.204003)
-        (xy 175.114609 100.204003)
-        (xy 175.114609 98.730803)
-        (xy 179.5272 98.730803)
+        (xy 182.937809 100.508803)
+        (xy 175.267009 100.508803)
+        (xy 175.267009 98.527603)
+        (xy 179.5272 98.527603)
         (xy 179.5272 97.9424)
       )
@@
       (pts
         (xy 168.1988 98.044)
-        (xy 168.2496 101.5492)
-        (xy 160.4264 101.5492)
-        (xy 160.4264 100.076)
-        (xy 164.846 100.076)
+        (xy 168.2496 101.7016)
+        (xy 160.4264 101.7016)
+        (xy 160.4264 99.0092)
+        (xy 164.846 99.0092)
         (xy 164.846 98.044)
       )
